Commit message: lskdjf

File: src/system_launch/models/tic_tac_toe_board.urdf (robot description, URDF)
Before this commit: robot tic_tac_toe_board_model, 1 links, 0 joints
Links:
- link tic_tac_toe_board: geometry collision mesh filename=package://system_launch/models/mesh/board_pieces.dae scale=.01 .01 .01; visual mesh filename=package://system_launch/models/mesh/board_pieces.dae scale=.01 .01 .01
