Commit message: update

File: src/system_launch/models/X.urdf (robot description, URDF)
Before this commit: robot X_model, 1 links, 0 joints
Links:
- link X: geometry collision mesh filename=package://system_launch/models/mesh/X_model.dae scale=0.008 0.008 0.008; visual mesh filename=package://system_launch/models/mesh/X_model.dae scale=0.008 0.008 0.008
