Commit message: pre presentation

File: src/system_launch/models/O.urdf (robot description, URDF)
Before this commit: robot O_model, 1 links, 0 joints
Links:
- link O: geometry collision mesh filename=package://system_launch/models/mesh/O_model.dae scale=.01 .01 .001; visual mesh filename=package://system_launch/models/mesh/O_model.dae scale=.01 .01 .001

File: src/system_launch/models/X.urdf (robot description, URDF)
Before this commit: robot X_model, 1 links, 0 joints
Links:
- link X: geometry collision mesh filename=package://system_launch/models/mesh/X_model.dae scale=0.008 0.008 0.001; visual mesh filename=package://system_launch/models/mesh/X_model.dae scale=0.008 0.008 0.001

File: src/system_launch/models/tic_tac_toe_board.urdf (robot description, URDF)
Before this commit: robot tic_tac_toe_board_model, 1 links, 0 joints
Links:
- link tic_tac_toe_board: geometry collision mesh filename=package://system_launch/models/mesh/board_pieces.dae scale=.01 .01 .001; visual mesh filename=package://system_launch/models/mesh/board_pieces.dae scale=.01 .01 .001
